File: layouts/default/default.kicad_pcb (KiCad board)
At the start: 2 copper layers, 108 parts

Commit message: Remove the 5A fuse
Parts:
- removed FH1: , XFCN_PTF_15:FUSE-TH_L22.0-W9.0-P22.60
- removed LED100, LED26, LED27, LED28, LED29, LED30, LED31, LED32, LED33, LED34, LED35, LED36, LED37, LED38, LED39, LED40, LED41, LED42, LED43, LED44, LED45, LED46, LED47, LED48, LED49, LED50, LED51, LED52, LED53, LED54, LED55, LED56, LED57, LED58, LED59, LED60, LED61, LED62, LED63, LED64, LED65, LED66, LED67, LED68, LED69, LED70, LED71, LED72, LED73, LED74, LED75, LED76, LED77, LED78, LED79, LED80, LED81, LED82, LED83, LED84, LED85, LED86, LED87, LED88, LED89, LED90, LED91, LED92, LED93, LED94, LED95, LED96, LED97, LED98, LED99: , XINGLIGHT_XL_5050RGBC_WS2812B:LED-SMD_4P-L5.0-W5.0-BL_XL-5050RGBC
- moved LED19 226.0 mm to (135.6, 104.2)
- moved LED22 223.9 mm to (123.0, 117.1)
- moved LED24 223.1 mm to (135.6, 117.1)
- moved LED17 211.1 mm to (123.0, 104.2)
- moved LED21 203.8 mm to (116.6, 117.1)
- moved LED10 201.7 mm to (141.9, 77.8)
- moved LED12 190.6 mm to (123.0, 90.4)
- moved LED9 189.9 mm to (135.6, 77.8)
- moved LED15 186.0 mm to (141.9, 90.4)
- moved LED13 185.9 mm to (129.3, 90.4)
- moved LED25 184.0 mm to (141.9, 117.1)
- moved LED20 181.4 mm to (141.9, 104.2)
- moved LED23 181.3 mm to (129.3, 117.1)
- moved LED7 174.6 mm to (123.0, 77.8)
- moved LED18 165.5 mm to (129.3, 104.2)
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Connections:
- net CC1 renamed A5
- C1 pad 2: VCC -> VDD
- LED1 pad 2: led_columns[0]-DOU-3 -> led_columns[0]-DIN-1
- LED1 pad 4: P1Y -> data_in
- LED10 pad 2: data_in-1 -> data_out
- LED10 pad 4: led_columns[0]-DIN-1 -> led_columns[1]-DIN-1
- LED11 pad 2: led_columns[1]-DOU-1 -> led_columns[2]-DOU
- LED11 pad 4: data_in-1 -> data_out
- LED12 pad 2: led_columns[1]-DIN-1 -> led_columns[2]-DIN
- LED12 pad 4: led_columns[1]-DOU-1 -> led_columns[2]-DOU
- LED13 pad 2: led_columns[1]-DOU-3 -> led_columns[2]-DIN-1
- LED13 pad 4: led_columns[1]-DIN-1 -> led_columns[2]-DIN
- LED14 pad 2: led_columns[1]-DIN-2 -> led_columns[2]-DOU-1
- LED14 pad 4: led_columns[1]-DOU-3 -> led_columns[2]-DIN-1
- LED15 pad 2: led_columns[1]-DOU-2 -> data_out-1
- LED15 pad 4: led_columns[1]-DIN-2 -> led_columns[2]-DOU-1
- LED16 pad 2: led_columns[1]-DIN-3 -> led_columns[3]-DOU-2
- LED16 pad 4: led_columns[1]-DOU-2 -> data_out-1
- LED17 pad 2: led_columns[1]-DOU-4 -> led_columns[3]-DOU
- LED17 pad 4: led_columns[1]-DIN-3 -> led_columns[3]-DOU-2
- LED18 pad 2: led_columns[1]-DIN -> led_columns[3]-DIN
- LED18 pad 4: led_columns[1]-DOU-4 -> led_columns[3]-DOU
- LED19 pad 2: led_columns[1]-DOU -> led_columns[3]-DOU-1
- LED19 pad 4: led_columns[1]-DIN -> led_columns[3]-DIN
- LED2 pad 2: led_columns[0]-DIN -> led_columns[0]-DOU
- LED2 pad 4: led_columns[0]-DOU-3 -> led_columns[0]-DIN-1
- LED20 pad 4: led_columns[1]-DOU -> led_columns[3]-DOU-1
- LED21 pad 2: led_columns[2]-DOU-2 -> led_columns[4]-DIN-2
- LED22 pad 2: led_columns[2]-DOU -> led_columns[4]-DOU
- LED22 pad 4: led_columns[2]-DOU-2 -> led_columns[4]-DIN-2
- LED23 pad 2: led_columns[2]-DIN -> led_columns[4]-DIN-1
- LED23 pad 4: led_columns[2]-DOU -> led_columns[4]-DOU
- LED24 pad 2: led_columns[2]-DOU-4 -> led_columns[4]-DIN
- LED24 pad 4: led_columns[2]-DIN -> led_columns[4]-DIN-1
- LED25 pad 2: led_columns[2]-DOU-1 -> led_columns[4]-data_out
- LED25 pad 4: led_columns[2]-DOU-4 -> led_columns[4]-DIN
- LED3 pad 2: led_columns[0]-DOU -> led_columns[0]-DIN-2
- LED3 pad 4: led_columns[0]-DIN -> led_columns[0]-DOU
- LED4 pad 2: led_columns[0]-DIN-3 -> led_columns[0]-DIN
- LED4 pad 4: led_columns[0]-DOU -> led_columns[0]-DIN-2
- LED5 pad 2: led_columns[0]-DOU-1 -> data_in-1
- LED5 pad 4: led_columns[0]-DIN-3 -> led_columns[0]-DIN
- LED6 pad 2: led_columns[0]-DIN-4 -> led_columns[1]-DIN
- LED6 pad 4: led_columns[0]-DOU-1 -> data_in-1
- LED7 pad 2: led_columns[0]-DOU-2 -> led_columns[1]-DIN-3
- LED7 pad 4: led_columns[0]-DIN-4 -> led_columns[1]-DIN
- LED8 pad 2: led_columns[0]-DIN-2 -> led_columns[1]-DIN-2
- LED8 pad 4: led_columns[0]-DOU-2 -> led_columns[1]-DIN-3
- LED9 pad 2: led_columns[0]-DIN-1 -> led_columns[1]-DIN-1
- LED9 pad 4: led_columns[0]-DIN-2 -> led_columns[1]-DIN-2
- R1 pad 1: P1Y -> data_in
- U2 pad 14: VCC -> VDD
- U2 pad 3: P1Y -> data_in
Routing:
- net VDD: track 0.00 -> 329.5 mm
- net gnd: track 0.00 -> 160.5 mm
- net data_in: track 0.00 -> 42.2 mm, vias 0 -> 2
- net data_out-1: track 0.00 -> 32.9 mm
- net data_out-2: track 0.00 -> 32.6 mm
- net data_in-1: track 0.00 -> 32.1 mm
- net data_out: track 0.00 -> 31.8 mm
- net EH: track 0.00 -> 16.3 mm
- net P1A: track 0.00 -> 14.0 mm
- net led_columns[2]-DOU-1: track 0.00 -> 6.38 mm
- net led_columns[4]-DIN: track 0.00 -> 6.38 mm
- net led_columns[3]-DOU-1: track 0.00 -> 6.38 mm
- net led_columns[1]-DIN-1: track 0.00 -> 6.38 mm
- net led_columns[0]-DIN: track 0.00 -> 6.38 mm
- net led_columns[2]-DOU: track 0.00 -> 6.38 mm
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- added copper zone on F.Cu, net gnd
Other:
- board outline added: 81.8 x 69.4 mm
