File: layouts/default/default.kicad_pcb (KiCad board)
At the start: 2 copper layers, 81.8 x 69.4 mm, 32 parts

Commit message: remove autogenerated trait, fix fp-lib-table, update gitignore
Connections:
- net data_in-2 renamed P1Y
- net data_in-4 renamed data_out-1
- net led_columns[1]-DOU-1 renamed led_columns[1]-DIN-1
- net led_columns[1]-DOU-2 renamed led_columns[1]-DIN-3
- net led_columns[2]-DOU-1 renamed led_columns[2]-DIN-1
- net led_columns[2]-DOU-2 renamed led_columns[2]-DIN-2
- net led_columns[3]-DIN renamed led_columns[3]-DOU-2
- LED1 pad 2: led_columns[0]-DOU -> led_columns[0]-DIN-1
- LED10 pad 4: led_columns[1]-DIN -> led_columns[1]-DIN-2
- LED15 pad 2: data_in-3 -> data_in-1
- LED16 pad 4: data_in-3 -> data_in-1
- LED18 pad 2: led_columns[3]-DOU -> led_columns[3]-DOU-3
- LED19 pad 2: led_columns[3]-DIN-1 -> led_columns[3]-DOU
- LED19 pad 4: led_columns[3]-DOU -> led_columns[3]-DOU-3
- LED2 pad 4: led_columns[0]-DOU -> led_columns[0]-DIN-1
- LED20 pad 2: data_in-1 -> data_in
- LED20 pad 4: led_columns[3]-DIN-1 -> led_columns[3]-DOU
- LED21 pad 2: led_columns[4]-DIN -> led_columns[4]-DOU-2
- LED21 pad 4: data_in-1 -> data_in
- LED22 pad 2: led_columns[4]-DOU -> led_columns[4]-DOU-3
- LED22 pad 4: led_columns[4]-DIN -> led_columns[4]-DOU-2
- LED23 pad 2: led_columns[4]-DOU-1 -> led_columns[4]-DOU
- LED23 pad 4: led_columns[4]-DOU -> led_columns[4]-DOU-3
- LED24 pad 2: led_columns[4]-DOU-2 -> led_columns[4]-DOU-1
- LED24 pad 4: led_columns[4]-DOU-1 -> led_columns[4]-DOU
- LED25 pad 2: data_out -> led_columns[4]-data_out
- LED25 pad 4: led_columns[4]-DOU-2 -> led_columns[4]-DOU-1
- LED3 pad 2: led_columns[0]-DIN-1 -> led_columns[0]-DOU
- LED4 pad 4: led_columns[0]-DIN-1 -> led_columns[0]-DOU
- LED5 pad 2: data_in -> data_out
- LED6 pad 2: led_columns[1]-DOU -> led_columns[1]-DIN
- LED6 pad 4: data_in -> data_out
- LED7 pad 4: led_columns[1]-DOU -> led_columns[1]-DIN
- LED9 pad 2: led_columns[1]-DIN -> led_columns[1]-DIN-2
Routing:
- net data_in-3: track 32.9 -> 0.00 mm
- net data_out: track 0.00 -> 32.1 mm
- net led_columns[3]-DIN-1: track 6.38 -> 0.00 mm
- net led_columns[1]-DIN-2: track 0.00 -> 6.38 mm
- net led_columns[4]-DOU-3: track 0.00 -> 6.38 mm
- net led_columns[4]-DIN: track 6.38 -> 0.00 mm
- net led_columns[1]-DOU: track 6.38 -> 0.00 mm
- net led_columns[3]-DOU-3: track 0.00 -> 6.38 mm
- net data_in: track 32.1 -> 32.6 mm
