File: layouts/default/default.kicad_pcb (KiCad board)
At the start: 2 copper layers, 81.8 x 69.4 mm, 32 parts

Commit message: Add pictures from the workshop
Connections:
- net data_in-1 renamed -data_out-3
- net data_in-3 renamed -data_out-2
- net data_in-4 renamed -data_out-1
- net data_out renamed led_columns[4]-data_out
- net led_columns[0]-DIN renamed led_columns[0]-DOU-3
- net led_columns[0]-DIN-1 renamed led_columns[0]-DOU-2
- net led_columns[0]-DOU renamed led_columns[0]-DOU-0
- net led_columns[1]-DIN renamed led_columns[1]-DOU-3
- net led_columns[1]-DOU renamed led_columns[1]-DOU-0
- net led_columns[2]-DOU renamed led_columns[2]-DOU-3
- net led_columns[3]-DIN-1 renamed led_columns[3]-DOU-3
- net led_columns[3]-DOU renamed led_columns[3]-DOU-2
- net led_columns[4]-DIN renamed led_columns[4]-DOU-0
- LED1 pad 4: data_in-2 -> data_in
- LED11 pad 2: led_columns[2]-DOU-1 -> led_columns[2]-DOU-0
- LED12 pad 2: led_columns[2]-DIN -> led_columns[2]-DOU-1
- LED12 pad 4: led_columns[2]-DOU-1 -> led_columns[2]-DOU-0
- LED13 pad 4: led_columns[2]-DIN -> led_columns[2]-DOU-1
- LED16 pad 2: led_columns[3]-DOU-1 -> led_columns[3]-DOU-0
- LED17 pad 2: led_columns[3]-DIN -> led_columns[3]-DOU-1
- LED17 pad 4: led_columns[3]-DOU-1 -> led_columns[3]-DOU-0
- LED18 pad 4: led_columns[3]-DIN -> led_columns[3]-DOU-1
- LED22 pad 2: led_columns[4]-DOU -> led_columns[4]-DOU-1
- LED23 pad 2: led_columns[4]-DOU-1 -> led_columns[4]-DOU-2
- LED23 pad 4: led_columns[4]-DOU -> led_columns[4]-DOU-1
- LED24 pad 2: led_columns[4]-DOU-2 -> led_columns[4]-DOU-3
- LED24 pad 4: led_columns[4]-DOU-1 -> led_columns[4]-DOU-2
- LED25 pad 4: led_columns[4]-DOU-2 -> led_columns[4]-DOU-3
- LED5 pad 2: data_in -> -data_out-0
- LED6 pad 4: data_in -> -data_out-0
- LED7 pad 2: led_columns[1]-DOU-2 -> led_columns[1]-DOU-1
- LED8 pad 2: led_columns[1]-DOU-1 -> led_columns[1]-DOU-2
- LED8 pad 4: led_columns[1]-DOU-2 -> led_columns[1]-DOU-1
- LED9 pad 4: led_columns[1]-DOU-1 -> led_columns[1]-DOU-2
- R1 pad 1: data_in-2 -> data_in
- U2 pad 3: data_in-2 -> data_in
Routing:
- net data_in-2: track 42.2 -> 0.00 mm, vias 2 -> 0
- net -data_out-0: track 0.00 -> 32.1 mm
- net data_in: track 32.1 -> 42.2 mm, vias 0 -> 2
- net led_columns[4]-DOU-3: track 0.00 -> 6.38 mm
- net led_columns[2]-DOU-0: track 0.00 -> 6.38 mm
- net led_columns[2]-DIN: track 6.38 -> 0.00 mm
- net led_columns[4]-DOU: track 6.38 -> 0.00 mm
- net led_columns[3]-DOU-0: track 0.00 -> 6.38 mm
- net led_columns[3]-DIN: track 6.38 -> 0.00 mm
