File: build/builds/default/default.20250618-163959.kicad_pcb (KiCad board)
At the start: 2 copper layers, 81.8 x 69.4 mm, 32 parts

Commit message: Add final board version
Connections:
- net data_in-3 renamed data_out-1
- net led_columns[1]-DOU-1 renamed led_columns[1]-DIN-2
- net led_columns[1]-DOU-2 renamed led_columns[1]-DIN-3
- net led_columns[2]-DOU-2 renamed led_columns[2]-DIN-1
- net led_columns[4]-DOU-1 renamed led_columns[4]-DIN-1
- C2 pad 1: P3V3 -> gnd
- C2 pad 2: gnd -> P3V3
- C3 pad 1: VDD -> gnd
- C3 pad 2: gnd -> VDD
- LED1 pad 2: led_columns[0]-DOU -> led_columns[0]-DIN-1
- LED1 pad 4: data_in-2 -> data_in
- LED10 pad 2: data_in-4 -> data_out
- LED10 pad 4: led_columns[1]-DIN -> led_columns[1]-DIN-1
- LED11 pad 2: led_columns[2]-DOU-1 -> led_columns[2]-DOU
- LED11 pad 4: data_in-4 -> data_out
- LED12 pad 4: led_columns[2]-DOU-1 -> led_columns[2]-DOU
- LED14 pad 2: led_columns[2]-DOU -> led_columns[2]-DOU-1
- LED15 pad 4: led_columns[2]-DOU -> led_columns[2]-DOU-1
- LED16 pad 2: led_columns[3]-DOU-1 -> led_columns[3]-DOU-2
- LED17 pad 2: led_columns[3]-DIN -> led_columns[3]-DOU
- LED17 pad 4: led_columns[3]-DOU-1 -> led_columns[3]-DOU-2
- LED18 pad 2: led_columns[3]-DOU -> led_columns[3]-DIN
- LED18 pad 4: led_columns[3]-DIN -> led_columns[3]-DOU
- LED19 pad 2: led_columns[3]-DIN-1 -> led_columns[3]-DOU-1
- LED19 pad 4: led_columns[3]-DOU -> led_columns[3]-DIN
- LED2 pad 2: led_columns[0]-DOU-1 -> led_columns[0]-DOU
- LED2 pad 4: led_columns[0]-DOU -> led_columns[0]-DIN-1
- LED20 pad 2: data_in-1 -> data_out-2
- LED20 pad 4: led_columns[3]-DIN-1 -> led_columns[3]-DOU-1
- LED21 pad 2: led_columns[4]-DIN -> led_columns[4]-DIN-2
- LED21 pad 4: data_in-1 -> data_out-2
- LED22 pad 4: led_columns[4]-DIN -> led_columns[4]-DIN-2
- LED24 pad 2: led_columns[4]-DOU-2 -> led_columns[4]-DIN
- LED25 pad 2: data_out -> led_columns[4]-data_out
- LED25 pad 4: led_columns[4]-DOU-2 -> led_columns[4]-DIN
- LED3 pad 2: led_columns[0]-DIN-1 -> led_columns[0]-DIN-2
- LED3 pad 4: led_columns[0]-DOU-1 -> led_columns[0]-DOU
- LED4 pad 4: led_columns[0]-DIN-1 -> led_columns[0]-DIN-2
- LED5 pad 2: data_in -> data_in-1
- LED6 pad 2: led_columns[1]-DOU -> led_columns[1]-DIN
- LED6 pad 4: data_in -> data_in-1
- LED7 pad 4: led_columns[1]-DOU -> led_columns[1]-DIN
- LED9 pad 2: led_columns[1]-DIN -> led_columns[1]-DIN-1
- R1 pad 1: data_in-2 -> data_in
- U2 pad 3: data_in-2 -> data_in
Routing:
- net data_in-2: track 42.2 -> 0.00 mm, vias 2 -> 0
- net data_out-2: track 0.00 -> 32.6 mm
- net data_out: track 0.00 -> 31.8 mm
- net data_in-4: track 31.8 -> 0.00 mm
- net data_in: track 32.1 -> 42.2 mm, vias 0 -> 2
- net led_columns[4]-DOU-2: track 6.38 -> 0.00 mm
- net led_columns[3]-DIN-1: track 6.38 -> 0.00 mm
- net led_columns[1]-DIN-1: track 0.00 -> 6.38 mm
- net led_columns[4]-DIN-2: track 0.00 -> 6.38 mm
- net led_columns[3]-DOU-2: track 0.00 -> 6.38 mm
- net led_columns[1]-DOU: track 6.38 -> 0.00 mm
- net led_columns[0]-DOU-1: track 6.38 -> 0.00 mm
- net led_columns[0]-DIN-2: track 0.00 -> 6.38 mm
- net gnd: track 165.1 -> 160.5 mm
- net P3V3: track 9.96 -> 5.61 mm
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Other:
- outline, holes or cut-outs redrawn
